File: pcb/LED matrix carrier/LED matrix.kicad_sch (KiCad schematic)
At the start: 10 parts, among them J1 Conn_01x15_Pin, J2 Conn_01x15_Socket, J3 Conn_01x02_Pin, J4 Conn_01x02_Socket, U1 74HC594, U2 74HC594, U3 74HC594

Commit message: fix wrong footprint/symbol
Parts:
- removed U1, U2, U3: 74HC594, Package_SO:TSSOP-16_4.4x5mm_P0.65mm, symbol 74xx:74HC594
- added U1, U2, U3: 74HC595, Package_SO:TSSOP-16_4.4x5mm_P0.65mm, symbol 74xx:74HC595
Connections:
- net +3V3: now also U1.10 (~{SRCLR}), U1.16 (VCC), U2.10 (~{SRCLR}), U2.16 (VCC), U3.10 (~{SRCLR}), U3.16 (VCC)
- net B0: now also U3.15 (QA)
- net B1: now also U3.1 (QB)
- net B2: now also U3.2 (QC)
- net B3: now also U3.3 (QD)
- net B4: now also U3.4 (QE)
- net B5: now also U3.5 (QF)
- net B6: now also U3.6 (QG)
- net B7: now also U3.7 (QH)
- net B_in: now also U3.14 (SER)
- net B_out: now also U3.9 (QH')
- net G0: now also U2.15 (QA)
- net G1: now also U2.1 (QB)
- net G2: now also U2.2 (QC)
- net G3: now also U2.3 (QD)
- net G4: now also U2.4 (QE)
- net G5: now also U2.5 (QF)
- net G6: now also U2.6 (QG)
- net G7: now also U2.7 (QH)
- net GND: now also U1.13 (~{OE}), U1.8 (GND), U2.13 (~{OE}), U2.8 (GND), U3.13 (~{OE}), U3.8 (GND)
- net G_in: now also U2.14 (SER)
- net G_out: now also U2.9 (QH')
- net R0: now also U1.15 (QA)
- net R1: now also U1.1 (QB)
- net R2: now also U1.2 (QC)
- net R3: now also U1.3 (QD)
- net R4: now also U1.4 (QE)
- net R5: now also U1.5 (QF)
- net R6: now also U1.6 (QG)
- net R7: now also U1.7 (QH)
- net RCLK: now also U1.12 (RCLK), U2.12 (RCLK), U3.12 (RCLK)
- net R_in: now also U1.14 (SER)
- net R_out: now also U1.9 (QH')
- net SRCLK: now also U1.11 (SRCLK), U2.11 (SRCLK), U3.11 (SRCLK)
