File: pcb/Carrier/Carrier.kicad_pcb (KiCad board)
At the start: 2 copper layers, 102.9 x 77.5 mm, 11 parts, among them J1 Conn_01x10_Pin, J2 Conn_01x10_Pin, J3 Conn_01x10_Pin, J4 Conn_01x10_Pin, J5 Conn_01x10_Pin, U1 ESP32-C6-DevKitC-1, U2 Tang_Nano_9k_board

Commit message: final design
Parts:
- added J6: Conn_01x16_Socket, Connector_PinSocket_2.54mm:PinSocket_1x16_P2.54mm_Vertical, B.Cu at (199.4, 96.5)
- added J7: Conn_01x16_Socket, Connector_PinSocket_2.54mm:PinSocket_1x16_P2.54mm_Vertical, B.Cu at (232.4, 96.5)
- moved REF** 7.62 mm to (229.9, 50.8)
- moved REF** 7.62 mm to (229.9, 118.1)
- moved U1 4.30 mm to (204.5, 96.5)
Connections:
- U1 pad 10: unconnected-(U1-GPIO10-Pad10) -> Net-(J6-Pin_10)
- U1 pad 11: unconnected-(U1-GPIO11-Pad11) -> Net-(J6-Pin_11)
- U1 pad 13: unconnected-(U1-GPIO3-Pad13) -> Net-(J6-Pin_13)
- U1 pad 14: unconnected-(U1-5V-Pad14) -> Net-(J6-Pin_14)
- U1 pad 19: unconnected-(U1-GPIO12/USB_D--Pad19) -> Net-(J7-Pin_14)
- U1 pad 2: unconnected-(U1-EN/RESET-Pad2) -> Net-(J6-Pin_2)
- U1 pad 20: unconnected-(U1-GPIO13/USB_D+-Pad20) -> Net-(J7-Pin_13)
- U1 pad 21: unconnected-(U1-GND-Pad21) -> GND
- U1 pad 22: unconnected-(U1-GPIO9/BOOT-Pad22) -> Net-(J7-Pin_11)
- U1 pad 23: unconnected-(U1-GPIO18-Pad23) -> Net-(J7-Pin_10)
- U1 pad 24: unconnected-(U1-GPIO19-Pad24) -> Net-(J7-Pin_9)
- U1 pad 25: unconnected-(U1-GPIO20-Pad25) -> Net-(J7-Pin_8)
- U1 pad 26: unconnected-(U1-GPIO21-Pad26) -> Net-(J7-Pin_7)
- U1 pad 27: unconnected-(U1-GPIO22-Pad27) -> Net-(J7-Pin_6)
- U1 pad 28: unconnected-(U1-GPIO23-Pad28) -> Net-(J7-Pin_5)
- U1 pad 29: unconnected-(U1-GPIO15/JTAG-Pad29) -> Net-(J7-Pin_4)
- U1 pad 3: unconnected-(U1-GPIO4/MTMS-Pad3) -> Net-(J6-Pin_3)
- U1 pad 30: unconnected-(U1-GPIO17/U0RXD-Pad30) -> Net-(J7-Pin_3)
- U1 pad 31: unconnected-(U1-GPIO16/U0TXD-Pad31) -> Net-(J7-Pin_2)
- U1 pad 7: unconnected-(U1-GPIO0-Pad7) -> Net-(J6-Pin_7)
- U1 pad 8: unconnected-(U1-GPIO1-Pad8) -> Net-(J6-Pin_8)
- U1 pad 9: unconnected-(U1-GPIO8/BOOT-Pad9) -> Net-(J6-Pin_9)
Routing:
- net +3V3: track 180.6 -> 120.5 mm
- net GND: track 70.2 -> 92.0 mm
- net Net-(J6-Pin_9): track 0.00 -> 5.08 mm
- net Net-(J6-Pin_8): track 0.00 -> 5.08 mm
- net Net-(J6-Pin_7): track 0.00 -> 5.08 mm
- net Net-(J6-Pin_3): track 0.00 -> 5.08 mm
- net Net-(J6-Pin_2): track 0.00 -> 5.08 mm
- net Net-(J6-Pin_14): track 0.00 -> 5.08 mm
- net Net-(J6-Pin_13): track 0.00 -> 5.08 mm
- net Net-(J6-Pin_11): track 0.00 -> 5.08 mm
- net Net-(J6-Pin_10): track 0.00 -> 5.08 mm
- net Net-(J7-Pin_9): track 0.00 -> 5.08 mm
- net Net-(J7-Pin_8): track 0.00 -> 5.08 mm
- net Net-(J7-Pin_7): track 0.00 -> 5.08 mm
- net Net-(J7-Pin_6): track 0.00 -> 5.08 mm
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- added copper zone on F.Cu, net +3V3
Other:
- board size 102.9 x 77.5 mm -> 110.5 x 77.5 mm
