File: pcb/Carrier/Carrier.kicad_sch (KiCad schematic)
At the start: 7 parts, among them J1 Conn_01x10_Pin, J2 Conn_01x10_Pin, J3 Conn_01x10_Pin, J4 Conn_01x10_Pin, J5 Conn_01x10_Pin, U1 ESP32-C6-DevKitC-1, U2 Tang_Nano_9k_board

Commit message: Change header pinout
Parts:
- J1, J2, J3, J4, J5: footprint Connector_PinHeader_2.54mm:PinHeader_1x10_P2.54mm_Horizontal -> Connector_PinHeader_2.54mm:PinHeader_1x10_P2.54mm_Vertical
Connections:
- net B0: now also J1.10 (Pin_10), U2.24 (69/IOT42A/RGB_G3/HDMI_CKP); no longer J1.7 (Pin_7), U2.22 (57/IOR13A/RGB_G5)
- net B1: now also J2.10 (Pin_10); no longer J2.7 (Pin_7)
- net B2: now also J3.10 (Pin_10); no longer J3.7 (Pin_7)
- net B3: now also J4.10 (Pin_10); no longer J4.7 (Pin_7)
- net B4: now also J5.10 (Pin_10); no longer J5.7 (Pin_7)
- net G0: now also J1.9 (Pin_9); no longer J1.6 (Pin_6)
- net G1: now also J2.9 (Pin_9); no longer J2.6 (Pin_6)
- net G2: now also J3.9 (Pin_9); no longer J3.6 (Pin_6)
- net G3: now also J4.9 (Pin_9); no longer J4.6 (Pin_6)
- net G4: now also J5.9 (Pin_9); no longer J5.6 (Pin_6)
- net GND: now also U2.26 (GND)
- net R0: now also J1.8 (Pin_8), U2.22 (57/IOR13A/RGB_G5); no longer J1.5 (Pin_5), U2.24 (69/IOT42A/RGB_G3/HDMI_CKP)
- net R1: now also J2.8 (Pin_8); no longer J2.5 (Pin_5)
- net R2: now also J3.8 (Pin_8); no longer J3.5 (Pin_5)
- net R3: now also J4.8 (Pin_8); no longer J4.5 (Pin_5)
- net R4: now also J5.8 (Pin_8); no longer J5.5 (Pin_5)
- net ROWSEL0: now also J1.5 (Pin_5), J2.5 (Pin_5), J3.5 (Pin_5), J4.5 (Pin_5), J5.5 (Pin_5); no longer J1.8 (Pin_8), J2.8 (Pin_8), J3.8 (Pin_8), J4.8 (Pin_8), J5.8 (Pin_8)
- net ROWSEL1: now also J1.6 (Pin_6), J2.6 (Pin_6), J3.6 (Pin_6), J4.6 (Pin_6), J5.6 (Pin_6); no longer J1.9 (Pin_9), J2.9 (Pin_9), J3.9 (Pin_9), J4.9 (Pin_9), J5.9 (Pin_9)
- net ROWSEL2: now also J1.7 (Pin_7), J2.7 (Pin_7), J3.7 (Pin_7), J4.7 (Pin_7), J5.7 (Pin_7); no longer J1.10 (Pin_10), J2.10 (Pin_10), J3.10 (Pin_10), J4.10 (Pin_10), J5.10 (Pin_10)

Commit message: Change FPGA Pin mapping
Connections:
- net RCLK: now also U2.6 (26/IOB8B); no longer U2.8 (28/IOB11B)
- net ROWSEL1: now also U2.8 (28/IOB11B); no longer U2.6 (26/IOB8B)
- net ROWSEL2: now also U2.9 (29/IOB13A); no longer U2.5 (25/IOB8A)
- net SRCLK: now also U2.5 (25/IOB8A); no longer U2.9 (29/IOB13A)
Changed lines of the file:
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@@
-		)
-	)
-	(label "ROWSEL2"
-		(at 113.03 72.39 180)
-		(effects
-			(font
-				(size 1.27 1.27)
-			)
-			(justify right bottom)
 		)
 	)
@@
 		)
 	)
+	(label "ROWSEL0"
+		(at 113.03 67.31 180)
+		(effects
+			(font
+				(size 1.27 1.27)
+			)
+			(justify right bottom)
+		)
+	)
 	(label "G1"
 		(at 182.88 43.18 0)
@@
 	)
 	(label "ROWSEL1"
-		(at 113.03 69.85 180)
+		(at 113.03 64.77 180)
 		(effects
 			(font
@@
 		)
 	)
-	(label "SRCLK"
-		(at 113.03 62.23 180)
-		(effects
-			(font
-				(size 1.27 1.27)
-			)
-			(justify right bottom)
-		)
-	)
 	(label "RCLK"
 		(at 33.02 106.68 0)
@@
 		)
 	)
+	(label "RCLK"
+		(at 113.03 69.85 180)
+		(effects
+			(font
+				(size 1.27 1.27)
+			)
+			(justify right bottom)
+		)
+	)
 	(label "SRCLK"
 		(at 33.02 104.14 0)
@@
 		)
 	)
-	(label "ROWSEL0"
-		(at 113.03 67.31 180)
-		(effects
-			(font
-				(size 1.27 1.27)
-			)
-			(justify right bottom)
-		)
-	)
 	(label "B1"
 		(at 182.88 40.64 0)
@@
 		)
 	)
-	(label "RCLK"
-		(at 113.03 64.77 180)
-		(effects
-			(font
+	(label "ROWSEL2"
+		(at 113.03 62.23 180)
+		(effects
+			(font
+				(size 1.27 1.27)
+			)
+			(justify right bottom)
+		)
+	)
+	(label "SRCLK"
+		(at 113.03 72.39 180)
+		(effects
+			(font

Commit message: final design
Parts:
- added J6, J7: Conn_01x16_Socket, Connector_PinSocket_2.54mm:PinSocket_1x16_P2.54mm_Vertical, symbol Connector:Conn_01x16_Socket
Connections:
- net +3V3: now also J6.1 (Pin_1)
- net GND: now also U1.21 (GND), J6.15 (Pin_15), J7.1 (Pin_1), J7.12 (Pin_12), J7.15 (Pin_15)
- net at U1.12 (GPIO2), U2.29 (49/IOR24A/SPILCD_RS): now also J6.12 (Pin_12)
- net at U1.6 (GPIO7), U2.35 (73/IOT39A/RGB_R5/HDMI_D1P): now also J6.6 (Pin_6)
- net at U1.5 (GPIO6), U2.36 (74/IOT38B/RGB_R4/HDMI_D2N): now also J6.5 (Pin_5)
- net at U1.4 (GPIO5/MTDI), U2.37 (75/IOT38A/RGB_R3/HDMI_D2P): now also J6.4 (Pin_4)
- net at U1.10 (GPIO10): now also J6.10 (Pin_10)
- net at U1.11 (GPIO11): now also J6.11 (Pin_11)
- net at U1.13 (GPIO3): now also J6.13 (Pin_13)
- net at U1.14 (5V): now also J6.14 (Pin_14)
- net at U1.19 (GPIO12/USB_D-): now also J7.14 (Pin_14)
- net at U1.2 (EN/RESET): now also J6.2 (Pin_2)
- net at U1.20 (GPIO13/USB_D+): now also J7.13 (Pin_13)
- net at U1.22 (GPIO9/BOOT): now also J7.11 (Pin_11)
- net at U1.23 (GPIO18): now also J7.10 (Pin_10)
- net at U1.24 (GPIO19): now also J7.9 (Pin_9)
- net at U1.25 (GPIO20): now also J7.8 (Pin_8)
- net at U1.26 (GPIO21): now also J7.7 (Pin_7)
- net at U1.27 (GPIO22): now also J7.6 (Pin_6)
- net at U1.28 (GPIO23): now also J7.5 (Pin_5)
- net at U1.29 (GPIO15/JTAG): now also J7.4 (Pin_4)
- net at U1.3 (GPIO4/MTMS): now also J6.3 (Pin_3)
- net at U1.30 (GPIO17/U0RXD): now also J7.3 (Pin_3)
- net at U1.31 (GPIO16/U0TXD): now also J7.2 (Pin_2)
- net at U1.7 (GPIO0): now also J6.7 (Pin_7)
- net at U1.8 (GPIO1): now also J6.8 (Pin_8)
- net at U1.9 (GPIO8/BOOT): now also J6.9 (Pin_9)
Other:
- moved on the sheet: U1, U2
